File: driver/driver.kicad_pcb (KiCad board)
At the start: 2 copper layers, 59 parts, among them J1 BARREL_JACK, J2 CONN_02X32, Q1 DUAL_NPN_MOSFET, Q10 DUAL_NPN_MOSFET, Q11 DUAL_NPN_MOSFET, Q12 DUAL_NPN_MOSFET, Q13 DUAL_NPN_MOSFET, Q14 DUAL_NPN_MOSFET, Q15 DUAL_NPN_MOSFET, Q16 DUAL_NPN_MOSFET, Q17 DUAL_NPN_MOSFET, Q18 DUAL_NPN_MOSFET, Q19 DUAL_NPN_MOSFET, Q2 DUAL_NPN_MOSFET, Q20 DUAL_NPN_MOSFET, Q21 DUAL_NPN_MOSFET, Q22 DUAL_NPN_MOSFET, Q23 DUAL_NPN_MOSFET, Q24 DUAL_NPN_MOSFET, Q25 DUAL_NPN_MOSFET, Q26 DUAL_NPN_MOSFET, Q27 DUAL_NPN_MOSFET, Q28 DUAL_NPN_MOSFET, Q29 DUAL_NPN_MOSFET, Q3 DUAL_NPN_MOSFET, Q30 DUAL_NPN_MOSFET, Q31 DUAL_NPN_MOSFET, Q32 DUAL_NPN_MOSFET, Q33 DUAL_NPN_MOSFET, Q34 DUAL_NPN_MOSFET, Q35 DUAL_NPN_MOSFET, Q36 DUAL_NPN_MOSFET, Q37 DUAL_NPN_MOSFET, Q38 DUAL_NPN_MOSFET, Q39 DUAL_NPN_MOSFET, Q4 DUAL_NPN_MOSFET, Q40 DUAL_NPN_MOSFET, Q41 DUAL_NPN_MOSFET, Q42 DUAL_NPN_MOSFET, Q43 DUAL_NPN_MOSFET, Q44 DUAL_NPN_MOSFET, Q5 DUAL_NPN_MOSFET, Q6 DUAL_NPN_MOSFET, Q7 DUAL_NPN_MOSFET, Q8 DUAL_NPN_MOSFET, Q9 DUAL_NPN_MOSFET, U1 MCP23017, U2 Teensy3.2, U3 MCP23017, U4 LM7815CT, U5 MCP23017, U6 LF50ABDT-TR, U7 MCP23017, U8 MCP23017, U9 MCP23017

Commit message: lots of revs
Parts:
- U1, U3, U5, U7: moved to B.Cu
- moved U1 118.4 mm to (123.2, 99.1)
- moved U3 62.0 mm to (178.1, 92.2)
- moved Q1 59.9 mm to (135.3, 114.3)
- moved Q4 52.4 mm to (135.3, 109.9)
- moved Q25 46.2 mm to (156.0, 114.4), turned to 180 degrees
- moved Q7 45.0 mm to (135.3, 105.4)
- moved Q28 40.9 mm to (156.0, 110.0), turned to 180 degrees
- moved Q44 37.9 mm to (156.0, 83.3), turned to 180 degrees
- moved Q10 37.7 mm to (135.3, 101.0)
- moved Q31 36.5 mm to (156.0, 105.5), turned to 180 degrees
- moved Q43 34.3 mm to (156.0, 87.8), turned to 180 degrees
- moved Q34 33.3 mm to (156.0, 101.1), turned to 180 degrees
- moved Q40 32.2 mm to (156.0, 92.2), turned to 180 degrees
- moved Q37 31.8 mm to (156.0, 96.6), turned to 180 degrees
- moved U5 31.5 mm to (121.9, 138.4)
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Connections:
- Q1 pad 4: /flipdot_matrix/R14+ -> /flipdot_matrix/FLIP+
- Q1 pad 6: /flipdot_matrix/FLIP+ -> /flipdot_matrix/R14+
- Q10 pad 4: /flipdot_matrix/R2+ -> /flipdot_matrix/FLIP+
- Q10 pad 6: /flipdot_matrix/FLIP+ -> /flipdot_matrix/R2+
- Q11 pad 4: /flipdot_matrix/FLIP+ -> GND
- Q11 pad 6: GND -> /flipdot_matrix/FLIP+
- Q12 pad 4: /flipdot_matrix/FLIP+ -> GND
- Q12 pad 6: GND -> /flipdot_matrix/FLIP+
- Q13 pad 4: /flipdot_matrix/R3+ -> /flipdot_matrix/FLIP+
- Q13 pad 6: /flipdot_matrix/FLIP+ -> /flipdot_matrix/R3+
- Q14 pad 4: /flipdot_matrix/FLIP+ -> GND
- Q14 pad 6: GND -> /flipdot_matrix/FLIP+
- Q15 pad 4: /flipdot_matrix/FLIP+ -> GND
- Q15 pad 6: GND -> /flipdot_matrix/FLIP+
- Q16 pad 4: /flipdot_matrix/R7+ -> /flipdot_matrix/FLIP+
- Q16 pad 6: /flipdot_matrix/FLIP+ -> /flipdot_matrix/R7+
- Q17 pad 4: /flipdot_matrix/FLIP+ -> GND
- Q17 pad 6: GND -> /flipdot_matrix/FLIP+
- Q18 pad 4: /flipdot_matrix/FLIP+ -> GND
- Q18 pad 6: GND -> /flipdot_matrix/FLIP+
- Q19 pad 4: /flipdot_matrix/R11+ -> /flipdot_matrix/FLIP+
- Q19 pad 6: /flipdot_matrix/FLIP+ -> /flipdot_matrix/R11+
- Q2 pad 4: /flipdot_matrix/FLIP+ -> GND
- Q2 pad 6: GND -> /flipdot_matrix/FLIP+
- Q20 pad 4: /flipdot_matrix/FLIP+ -> GND
- Q20 pad 6: GND -> /flipdot_matrix/FLIP+
- Q21 pad 4: /flipdot_matrix/FLIP+ -> GND
- Q21 pad 6: GND -> /flipdot_matrix/FLIP+
- Q22 pad 4: /flipdot_matrix/R15+ -> /flipdot_matrix/FLIP+
- Q22 pad 6: /flipdot_matrix/FLIP+ -> /flipdot_matrix/R15+
- Q23 pad 4: /flipdot_matrix/FLIP+ -> GND
- Q23 pad 6: GND -> /flipdot_matrix/FLIP+
- Q24 pad 4: /flipdot_matrix/FLIP+ -> GND
- Q24 pad 6: GND -> /flipdot_matrix/FLIP+
- Q25 pad 4: GND -> /flipdot_matrix/R14-
- Q25 pad 6: /flipdot_matrix/R14- -> GND
- Q26 pad 4: /flipdot_matrix/FLIP+ -> GND
- Q26 pad 6: GND -> /flipdot_matrix/FLIP+
- Q27 pad 4: /flipdot_matrix/FLIP+ -> GND
- Q27 pad 6: GND -> /flipdot_matrix/FLIP+
- Q28 pad 4: GND -> /flipdot_matrix/R10-
- Q28 pad 6: /flipdot_matrix/R10- -> GND
- Q29 pad 4: /flipdot_matrix/FLIP+ -> GND
- Q29 pad 6: GND -> /flipdot_matrix/FLIP+
- Q3 pad 4: /flipdot_matrix/FLIP+ -> GND
- Q3 pad 6: GND -> /flipdot_matrix/FLIP+
- Q30 pad 4: /flipdot_matrix/FLIP+ -> GND
- Q30 pad 6: GND -> /flipdot_matrix/FLIP+
- Q31 pad 4: GND -> /flipdot_matrix/R6-
- Q31 pad 6: /flipdot_matrix/R6- -> GND
- Q32 pad 4: /flipdot_matrix/FLIP+ -> GND
- Q32 pad 6: GND -> /flipdot_matrix/FLIP+
- Q33 pad 4: /flipdot_matrix/FLIP+ -> GND
- Q33 pad 6: GND -> /flipdot_matrix/FLIP+
- Q34 pad 4: GND -> /flipdot_matrix/R2-
- Q34 pad 6: /flipdot_matrix/R2- -> GND
- Q35 pad 4: /flipdot_matrix/FLIP+ -> GND
- Q35 pad 6: GND -> /flipdot_matrix/FLIP+
- Q36 pad 4: /flipdot_matrix/FLIP+ -> GND
- Q36 pad 6: GND -> /flipdot_matrix/FLIP+
- Q37 pad 4: GND -> /flipdot_matrix/R3-
- Q37 pad 6: /flipdot_matrix/R3- -> GND
- Q38 pad 4: /flipdot_matrix/FLIP+ -> GND
- Q38 pad 6: GND -> /flipdot_matrix/FLIP+
- Q39 pad 4: /flipdot_matrix/FLIP+ -> GND
- Q39 pad 6: GND -> /flipdot_matrix/FLIP+
- Q4 pad 4: /flipdot_matrix/R10+ -> /flipdot_matrix/FLIP+
- Q4 pad 6: /flipdot_matrix/FLIP+ -> /flipdot_matrix/R10+
- Q40 pad 4: GND -> /flipdot_matrix/R7-
- Q40 pad 6: /flipdot_matrix/R7- -> GND
- Q41 pad 4: /flipdot_matrix/FLIP+ -> GND
- Q41 pad 6: GND -> /flipdot_matrix/FLIP+
- Q42 pad 4: /flipdot_matrix/FLIP+ -> GND
- Q42 pad 6: GND -> /flipdot_matrix/FLIP+
- Q43 pad 4: GND -> /flipdot_matrix/R11-
- Q43 pad 6: /flipdot_matrix/R11- -> GND
- Q44 pad 4: GND -> /flipdot_matrix/R15-
- Q44 pad 6: /flipdot_matrix/R15- -> GND
- Q5 pad 4: /flipdot_matrix/FLIP+ -> GND
- Q5 pad 6: GND -> /flipdot_matrix/FLIP+
- Q6 pad 4: /flipdot_matrix/FLIP+ -> GND
- Q6 pad 6: GND -> /flipdot_matrix/FLIP+
- Q7 pad 4: /flipdot_matrix/R6+ -> /flipdot_matrix/FLIP+
- Q7 pad 6: /flipdot_matrix/FLIP+ -> /flipdot_matrix/R6+
- Q8 pad 4: /flipdot_matrix/FLIP+ -> GND
- Q8 pad 6: GND -> /flipdot_matrix/FLIP+
- Q9 pad 4: /flipdot_matrix/FLIP+ -> GND
- Q9 pad 6: GND -> /flipdot_matrix/FLIP+
- U1 pad 2: /flipdot_matrix/ROW1- -> /flipdot_matrix/ROW3+
- U1 pad 21: /flipdot_matrix/ROW5+ -> /flipdot_matrix/ROW2+
- U1 pad 22: /flipdot_matrix/ROW5- -> /flipdot_matrix/ROW4+
- U1 pad 24: /flipdot_matrix/ROW6- -> /flipdot_matrix/ROW8+
- U1 pad 25: /flipdot_matrix/ROW7+ -> /flipdot_matrix/ROW10+
- U1 pad 26: /flipdot_matrix/ROW7- -> /flipdot_matrix/ROW12+
- U1 pad 27: /flipdot_matrix/ROW8+ -> /flipdot_matrix/ROW14+
- U1 pad 28: /flipdot_matrix/ROW8- -> /flipdot_matrix/ROW16+
- U1 pad 3: /flipdot_matrix/ROW2+ -> /flipdot_matrix/ROW5+
- U1 pad 4: /flipdot_matrix/ROW2- -> /flipdot_matrix/ROW7+
- U1 pad 5: /flipdot_matrix/ROW3+ -> /flipdot_matrix/ROW9+
- U1 pad 6: /flipdot_matrix/ROW3- -> /flipdot_matrix/ROW11+
- U1 pad 7: /flipdot_matrix/ROW4+ -> /flipdot_matrix/ROW13+
- U1 pad 8: /flipdot_matrix/ROW4- -> /flipdot_matrix/ROW15+
- U3 pad 1: /flipdot_matrix/ROW9+ -> /flipdot_matrix/ROW15-
- U3 pad 2: /flipdot_matrix/ROW9- -> /flipdot_matrix/ROW13-
- U3 pad 21: /flipdot_matrix/ROW13+ -> /flipdot_matrix/ROW2-
- U3 pad 22: /flipdot_matrix/ROW13- -> /flipdot_matrix/ROW4-
- U3 pad 23: /flipdot_matrix/ROW14+ -> /flipdot_matrix/ROW6-
- U3 pad 24: /flipdot_matrix/ROW14- -> /flipdot_matrix/ROW8-
- U3 pad 25: /flipdot_matrix/ROW15+ -> /flipdot_matrix/ROW10-
- U3 pad 26: /flipdot_matrix/ROW15- -> /flipdot_matrix/ROW12-
- U3 pad 27: /flipdot_matrix/ROW16+ -> /flipdot_matrix/ROW14-
- U3 pad 3: /flipdot_matrix/ROW10+ -> /flipdot_matrix/ROW11-
- U3 pad 4: /flipdot_matrix/ROW10- -> /flipdot_matrix/ROW9-
- U3 pad 5: /flipdot_matrix/ROW11+ -> /flipdot_matrix/ROW7-
- U3 pad 6: /flipdot_matrix/ROW11- -> /flipdot_matrix/ROW5-
- U3 pad 7: /flipdot_matrix/ROW12+ -> /flipdot_matrix/ROW3-
- U3 pad 8: /flipdot_matrix/ROW12- -> /flipdot_matrix/ROW1-
- U5 pad 1: /flipdot_matrix/COL1+ -> /flipdot_matrix/COL7-
- U5 pad 2: /flipdot_matrix/COL1- -> /flipdot_matrix/COL7+
- U5 pad 3: /flipdot_matrix/COL3+ -> /flipdot_matrix/COL5-
- U5 pad 4: /flipdot_matrix/COL3- -> /flipdot_matrix/COL5+
- U5 pad 5: /flipdot_matrix/COL5+ -> /flipdot_matrix/COL3+
- U5 pad 6: /flipdot_matrix/COL5- -> /flipdot_matrix/COL3-
- U5 pad 7: /flipdot_matrix/COL7+ -> /flipdot_matrix/COL1+
- U5 pad 8: /flipdot_matrix/COL7- -> /flipdot_matrix/COL1-
- U7 pad 1: /flipdot_matrix/COL17+ -> /flipdot_matrix/COL25+
- U7 pad 2: /flipdot_matrix/COL17- -> /flipdot_matrix/COL25-
- U7 pad 21: /flipdot_matrix/COL25+ -> /flipdot_matrix/COL17+
- U7 pad 22: /flipdot_matrix/COL25- -> /flipdot_matrix/COL17-
- U7 pad 23: /flipdot_matrix/COL27+ -> /flipdot_matrix/COL19+
- U7 pad 24: /flipdot_matrix/COL27- -> /flipdot_matrix/COL19-
- U7 pad 25: Net-(U7-Pad25) -> /flipdot_matrix/COL21+
- U7 pad 26: Net-(U7-Pad26) -> /flipdot_matrix/COL21-
- U7 pad 3: /flipdot_matrix/COL19+ -> /flipdot_matrix/COL27+
- U7 pad 4: /flipdot_matrix/COL19- -> /flipdot_matrix/COL27-
- U7 pad 5: /flipdot_matrix/COL21+ -> Net-(U7-Pad5)
- U7 pad 6: /flipdot_matrix/COL21- -> Net-(U7-Pad6)
Routing:
- net GND: track 225.3 -> 365.4 mm, vias 28 -> 0
- net /flipdot_matrix/ROW15+: track 0.00 -> 30.6 mm, vias 0 -> 1
- net /flipdot_matrix/ROW3+: track 0.00 -> 30.4 mm, vias 0 -> 1
- net /flipdot_matrix/ROW11+: track 0.00 -> 29.8 mm, vias 0 -> 1
- net /flipdot_matrix/ROW7+: track 0.00 -> 28.9 mm, vias 0 -> 1
- net /flipdot_matrix/COL1+: track 4.53 -> 31.7 mm
- net /flipdot_matrix/COL3+: track 4.41 -> 30.1 mm
- net /flipdot_matrix/COL7+: track 4.35 -> 29.9 mm
- net /flipdot_matrix/ROW1+: track 0.00 -> 25.5 mm, vias 0 -> 1
- net /flipdot_matrix/COL5+: track 4.53 -> 29.8 mm
- net /flipdot_matrix/ROW13+: track 0.00 -> 25.0 mm, vias 0 -> 1
- net /flipdot_matrix/ROW9+: track 0.00 -> 24.1 mm, vias 0 -> 1
- net /flipdot_matrix/COL1-: track 2.11 -> 25.5 mm
- net /flipdot_matrix/ROW5+: track 0.00 -> 23.1 mm, vias 0 -> 1
- net /flipdot_matrix/ROW14+: track 0.00 -> 22.7 mm, vias 0 -> 1
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Other:
- net class FLIP: clearance 0.25 -> 0.2
