File: driver/driver.kicad_pcb (KiCad board)
At the start: 2 copper layers, 59 parts, among them J1 BARREL_JACK, J2 CONN_02X32, Q1 DUAL_NPN_MOSFET, Q10 DUAL_NPN_MOSFET, Q11 DUAL_NPN_MOSFET, Q12 DUAL_NPN_MOSFET, Q13 DUAL_NPN_MOSFET, Q14 DUAL_NPN_MOSFET, Q15 DUAL_NPN_MOSFET, Q16 DUAL_NPN_MOSFET, Q17 DUAL_NPN_MOSFET, Q18 DUAL_NPN_MOSFET, Q19 DUAL_NPN_MOSFET, Q2 DUAL_NPN_MOSFET, Q20 DUAL_NPN_MOSFET, Q21 DUAL_NPN_MOSFET, Q22 DUAL_NPN_MOSFET, Q23 DUAL_NPN_MOSFET, Q24 DUAL_NPN_MOSFET, Q25 DUAL_NPN_MOSFET, Q26 DUAL_NPN_MOSFET, Q27 DUAL_NPN_MOSFET, Q28 DUAL_NPN_MOSFET, Q29 DUAL_NPN_MOSFET, Q3 DUAL_NPN_MOSFET, Q30 DUAL_NPN_MOSFET, Q31 DUAL_NPN_MOSFET, Q32 DUAL_NPN_MOSFET, Q33 DUAL_NPN_MOSFET, Q34 DUAL_NPN_MOSFET, Q35 DUAL_NPN_MOSFET, Q36 DUAL_NPN_MOSFET, Q37 DUAL_NPN_MOSFET, Q38 DUAL_NPN_MOSFET, Q39 DUAL_NPN_MOSFET, Q4 DUAL_NPN_MOSFET, Q40 DUAL_NPN_MOSFET, Q41 DUAL_NPN_MOSFET, Q42 DUAL_NPN_MOSFET, Q43 DUAL_NPN_MOSFET, Q44 DUAL_NPN_MOSFET, Q5 DUAL_NPN_MOSFET, Q6 DUAL_NPN_MOSFET, Q7 DUAL_NPN_MOSFET, Q8 DUAL_NPN_MOSFET, Q9 DUAL_NPN_MOSFET, U1 MCP23017, U2 Teensy3.2, U3 MCP23017, U4 LM7815CT, U5 MCP23017, U6 LF50ABDT-TR, U7 MCP23017, U8 MCP23017, U9 MCP23017

Commit message: closer to final
Parts:
- added G***: LOGO, img:flipdot, F.Cu at (124.5, 124.5)
- added G***: LOGO, img:driver, F.Cu at (169.5, 125.1)
- added J3: CONN_01X04, Pin_Headers:Pin_Header_Straight_1x04_Pitch2.54mm, F.Cu at (122.6, 79.4)
- added REF**: MountingHole_2.2mm_M2, Mounting_Holes:MountingHole_2.2mm_M2, F.Cu at (122.7, 177.0)
- added REF**: MountingHole_2.2mm_M2, Mounting_Holes:MountingHole_2.2mm_M2, F.Cu at (168.9, 177.0)
- C1, C2: footprint Capacitors_THT:CP_Radial_Tantal_D10.5mm_P5.00mm -> Capacitors_SMD:C_0805_HandSoldering
- C3: value 10uF -> 22uF; footprint Capacitors_THT:CP_Radial_Tantal_D10.5mm_P5.00mm -> Capacitors_SMD:C_0805_HandSoldering
- Q1, Q10, Q11, Q12, Q13, Q14, Q15, Q16, Q17, Q18, Q19, Q2, Q20, Q21, Q22, Q23, Q24, Q25, Q26, Q27, Q28, Q29, Q3, Q30, Q31, Q32, Q33, Q34, Q35, Q36, Q37, Q38, Q39, Q4, Q40, Q41, Q42, Q43, Q44, Q5, Q6, Q7, Q8, Q9: footprint TO_SOT_Packages_SMD:SOT-363_SC-70-6_Handsoldering -> TO_SOT_Packages_SMD:SOT-23-6_Handsoldering
- R1: footprint Resistors_THT:R_Axial_DIN0204_L3.6mm_D1.6mm_P7.62mm_Horizontal -> Resistors_THT:R_Axial_DIN0414_L11.9mm_D4.5mm_P15.24mm_Horizontal
- U8, U9: moved to B.Cu
- moved U6 106.6 mm to (167.1, 79.8), turned to 270 degrees
- moved R1 86.6 mm to (128.3, 77.5)
- moved J1 85.4 mm to (167.6, 66.0)
- moved U4 81.0 mm to (153.9, 77.7)
- moved C2 78.6 mm to (166.1, 73.4)
- moved C3 75.8 mm to (148.1, 78.2), turned to 90 degrees
- moved C1 56.1 mm to (169.9, 72.4), turned to 270 degrees
- moved U2 51.7 mm to (138.7, 64.3), turned to 0 degrees
- moved U9 33.9 mm to (172.5, 166.5)
- moved U8 28.3 mm to (173.2, 131.1)
- moved Q42 24.1 mm to (148.6, 176.5), turned to 270 degrees
- moved Q30 22.6 mm to (157.5, 176.5), turned to 270 degrees
- moved Q36 22.4 mm to (153.0, 176.5), turned to 270 degrees
- moved Q12 21.1 mm to (158.9, 160.4)
- moved Q24 21.1 mm to (158.9, 170.6)
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Connections:
- net Net-(C1-Pad1) renamed /JACK_IN
- U7 pad 1: /flipdot_matrix/COL25+ -> /flipdot_matrix/COL23+
- U7 pad 2: /flipdot_matrix/COL25- -> /flipdot_matrix/COL23-
- U7 pad 3: /flipdot_matrix/COL27+ -> /flipdot_matrix/COL25+
- U7 pad 4: /flipdot_matrix/COL27- -> /flipdot_matrix/COL25-
- U7 pad 7: /flipdot_matrix/COL23+ -> /flipdot_matrix/COL27+
- U7 pad 8: /flipdot_matrix/COL23- -> /flipdot_matrix/COL27-
- U8 pad 1: /flipdot_matrix/COL2+ -> /flipdot_matrix/COL8+
- U8 pad 2: /flipdot_matrix/COL2- -> /flipdot_matrix/COL8-
- U8 pad 3: /flipdot_matrix/COL4+ -> /flipdot_matrix/COL6+
- U8 pad 4: /flipdot_matrix/COL4- -> /flipdot_matrix/COL6-
- U8 pad 5: /flipdot_matrix/COL6+ -> /flipdot_matrix/COL4+
- U8 pad 6: /flipdot_matrix/COL6- -> /flipdot_matrix/COL4-
- U8 pad 7: /flipdot_matrix/COL8+ -> /flipdot_matrix/COL2+
- U8 pad 8: /flipdot_matrix/COL8- -> /flipdot_matrix/COL2-
- U9 pad 1: /flipdot_matrix/COL18+ -> /flipdot_matrix/COL28+
- U9 pad 2: /flipdot_matrix/COL18- -> /flipdot_matrix/COL28-
- U9 pad 21: /flipdot_matrix/COL26+ -> /flipdot_matrix/COL26-
- U9 pad 22: /flipdot_matrix/COL26- -> /flipdot_matrix/COL26+
- U9 pad 23: /flipdot_matrix/COL28+ -> /flipdot_matrix/COL24-
- U9 pad 24: /flipdot_matrix/COL28- -> /flipdot_matrix/COL24+
- U9 pad 3: /flipdot_matrix/COL20+ -> /flipdot_matrix/COL22-
- U9 pad 4: /flipdot_matrix/COL20- -> /flipdot_matrix/COL22+
- U9 pad 5: /flipdot_matrix/COL22+ -> /flipdot_matrix/COL20-
- U9 pad 6: /flipdot_matrix/COL22- -> /flipdot_matrix/COL20+
- U9 pad 7: /flipdot_matrix/COL24+ -> /flipdot_matrix/COL18-
- U9 pad 8: /flipdot_matrix/COL24- -> /flipdot_matrix/COL18+
Routing:
- net GND: track 365.4 -> 544.8 mm, vias 0 -> 2
- net VCC: track 6.02 -> 66.1 mm, vias 0 -> 1
- net /flipdot_matrix/FLIP+: track 302.7 -> 340.5 mm
- net /SDA: track 0.00 -> 37.4 mm
- net /JACK_IN: track 0.00 -> 34.8 mm
- net /flipdot_matrix/COL16+: track 0.00 -> 34.2 mm, vias 0 -> 1
- net /flipdot_matrix/COL27+: track 1.08 -> 35.1 mm, vias 0 -> 1
- net /flipdot_matrix/ROW14-: track 0.00 -> 33.7 mm, vias 0 -> 1
- net /SCL: track 0.00 -> 33.5 mm
- net /flipdot_matrix/COL26+: track 0.00 -> 33.2 mm, vias 0 -> 1
- net /flipdot_matrix/COL14+: track 0.00 -> 31.8 mm, vias 0 -> 1
- net /flipdot_matrix/ROW10-: track 0.00 -> 30.9 mm, vias 0 -> 1
- net /flipdot_matrix/COL12+: track 0.00 -> 30.4 mm, vias 0 -> 1
- net /flipdot_matrix/COL16-: track 0.00 -> 29.3 mm, vias 0 -> 1
- net /flipdot_matrix/COL10+: track 0.00 -> 29.2 mm, vias 0 -> 1
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Other:
- net class real hours added: clearance 0.4, trace_width 0.65, via_dia 0.6, via_drill 0.4
- net class thicc added: clearance 0.25, trace_width 0.45, via_dia 0.6, via_drill 0.4

Commit message: wild changes
Parts:
- moved U5 3.02 mm to (124.7, 139.6)
- moved U7 2.79 mm to (124.7, 162.2)
- moved U1 1.61 mm to (124.7, 99.6)
Routing:
- net VCC: track 66.1 -> 118.5 mm, vias 1 -> 4
- net GND: track 544.8 -> 574.6 mm, vias 2 -> 5
- net /SCL: track 33.5 -> 52.3 mm, vias 0 -> 1
- net /SDA: track 37.4 -> 49.9 mm
- net /flipdot_matrix/COL7-: track 23.3 -> 30.9 mm, vias 1 -> 3
- net /flipdot_matrix/COL7+: track 29.9 -> 35.3 mm, vias 1 -> 3
- net /flipdot_matrix/COL25-: track 27.8 -> 24.0 mm
- net /flipdot_matrix/COL25+: track 29.1 -> 25.4 mm
- net /flipdot_matrix/COL23+: track 24.7 -> 21.0 mm
- net /flipdot_matrix/COL27+: track 35.1 -> 31.5 mm
- net /flipdot_matrix/COL27-: track 31.7 -> 28.3 mm
- net /flipdot_matrix/COL23-: track 23.2 -> 19.8 mm
- net /flipdot_matrix/COL9-: track 7.35 -> 4.08 mm
- net /flipdot_matrix/COL11+: track 15.7 -> 12.5 mm
- net /flipdot_matrix/COL5-: track 23.1 -> 26.3 mm
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
Commit message: done??
probably not
Parts:
- removed G***: LOGO, img:flipdot
- removed G***: LOGO, img:driver
- removed J2: CONN_02X32, Socket_Strips:Socket_Strip_Straight_2x32_Pitch2.54mm
- removed REF** (x2): MountingHole_2.2mm_M2, Mounting_Holes:MountingHole_2.2mm_M2
- added J10: C96ABC, img:C96ABCMD_custom, F.Cu at (148.1, 83.8)
- added R2: 4.7k, Resistors_SMD:R_0805_HandSoldering, F.Cu at (126.5, 66.0)
- added R3: 4.7k, Resistors_SMD:R_0805_HandSoldering, F.Cu at (134.9, 68.1)
- moved U8 5.58 mm to (168.4, 128.3)
- moved U9 3.81 mm to (168.7, 166.5)
Connections:
- U7 pad 15: GND -> VCC
- U8 pad 16: VCC -> GND
- U8 pad 17: GND -> VCC
- U9 pad 15: GND -> VCC
- U9 pad 16: VCC -> GND
- U9 pad 17: GND -> VCC
Routing:
- net VCC: track 118.5 -> 382.0 mm, vias 4 -> 12
- net /SCL: track 52.3 -> 268.5 mm, vias 1 -> 6
- net /SDA: track 49.9 -> 260.5 mm, vias 0 -> 6
- net GND: track 574.6 -> 644.1 mm, vias 5 -> 10
- net /flipdot_matrix/FLIP+: track 340.5 -> 352.0 mm, vias 28 -> 29
- net /flipdot_matrix/COL2+: track 26.3 -> 17.9 mm
- net /flipdot_matrix/COL2-: track 19.5 -> 11.6 mm
- net /flipdot_matrix/COL4-: track 15.8 -> 7.83 mm
- net /flipdot_matrix/COL4+: track 22.1 -> 14.2 mm
- net /flipdot_matrix/COL6-: track 11.7 -> 4.85 mm
- net /flipdot_matrix/COL6+: track 17.9 -> 11.5 mm
- net /flipdot_matrix/COL24+: track 27.3 -> 23.4 mm
- net /flipdot_matrix/COL24-: track 23.6 -> 19.8 mm
- net /flipdot_matrix/COL28+: track 27.9 -> 24.1 mm
- net /flipdot_matrix/COL26-: track 28.7 -> 24.9 mm
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
Commit message: fix major goof
Parts:
- added G***: LOGO, img:flipdot, F.Cu at (125.1, 127.6)
- added G***: LOGO, img:driver, F.Cu at (168.3, 127.6)
- C3: footprint Capacitors_SMD:C_0805_HandSoldering -> Resistors_SMD:R_1206_HandSoldering
- moved C3 0.92 mm to (147.3, 77.7)
Connections:
- Q1 pad 1: /flipdot_matrix/FLIP+ -> /flipdot_matrix/R14+
- Q1 pad 2: /flipdot_matrix/ROW16+ -> /flipdot_matrix/ROW14+
- Q1 pad 3: /flipdot_matrix/R16+ -> /flipdot_matrix/FLIP+
- Q1 pad 4: /flipdot_matrix/FLIP+ -> /flipdot_matrix/R16+
- Q1 pad 5: /flipdot_matrix/ROW14+ -> /flipdot_matrix/ROW16+
- Q1 pad 6: /flipdot_matrix/R14+ -> /flipdot_matrix/FLIP+
- Q10 pad 1: /flipdot_matrix/FLIP+ -> /flipdot_matrix/R2+
- Q10 pad 2: /flipdot_matrix/ROW4+ -> /flipdot_matrix/ROW2+
- Q10 pad 3: /flipdot_matrix/R4+ -> /flipdot_matrix/FLIP+
- Q10 pad 4: /flipdot_matrix/FLIP+ -> /flipdot_matrix/R4+
- Q10 pad 5: /flipdot_matrix/ROW2+ -> /flipdot_matrix/ROW4+
- Q10 pad 6: /flipdot_matrix/R2+ -> /flipdot_matrix/FLIP+
- Q13 pad 1: /flipdot_matrix/FLIP+ -> /flipdot_matrix/R3+
- Q13 pad 2: /flipdot_matrix/ROW1+ -> /flipdot_matrix/ROW3+
- Q13 pad 3: /flipdot_matrix/R1+ -> /flipdot_matrix/FLIP+
- Q13 pad 4: /flipdot_matrix/FLIP+ -> /flipdot_matrix/R1+
- Q13 pad 5: /flipdot_matrix/ROW3+ -> /flipdot_matrix/ROW1+
- Q13 pad 6: /flipdot_matrix/R3+ -> /flipdot_matrix/FLIP+
- Q16 pad 1: /flipdot_matrix/FLIP+ -> /flipdot_matrix/R7+
- Q16 pad 2: /flipdot_matrix/ROW5+ -> /flipdot_matrix/ROW7+
- Q16 pad 3: /flipdot_matrix/R5+ -> /flipdot_matrix/FLIP+
- Q16 pad 4: /flipdot_matrix/FLIP+ -> /flipdot_matrix/R5+
- Q16 pad 5: /flipdot_matrix/ROW7+ -> /flipdot_matrix/ROW5+
- Q16 pad 6: /flipdot_matrix/R7+ -> /flipdot_matrix/FLIP+
- Q19 pad 1: /flipdot_matrix/FLIP+ -> /flipdot_matrix/R11+
- Q19 pad 2: /flipdot_matrix/ROW9+ -> /flipdot_matrix/ROW11+
- Q19 pad 3: /flipdot_matrix/R9+ -> /flipdot_matrix/FLIP+
- Q19 pad 4: /flipdot_matrix/FLIP+ -> /flipdot_matrix/R9+
- Q19 pad 5: /flipdot_matrix/ROW11+ -> /flipdot_matrix/ROW9+
- Q19 pad 6: /flipdot_matrix/R11+ -> /flipdot_matrix/FLIP+
- Q22 pad 1: /flipdot_matrix/FLIP+ -> /flipdot_matrix/R15+
- Q22 pad 2: /flipdot_matrix/ROW13+ -> /flipdot_matrix/ROW15+
- Q22 pad 3: /flipdot_matrix/R13+ -> /flipdot_matrix/FLIP+
- Q22 pad 4: /flipdot_matrix/FLIP+ -> /flipdot_matrix/R13+
- Q22 pad 5: /flipdot_matrix/ROW15+ -> /flipdot_matrix/ROW13+
- Q22 pad 6: /flipdot_matrix/R15+ -> /flipdot_matrix/FLIP+
- Q25 pad 1: /flipdot_matrix/R16- -> GND
- Q25 pad 2: /flipdot_matrix/ROW16- -> /flipdot_matrix/ROW14-
- Q25 pad 3: GND -> /flipdot_matrix/R14-
- Q25 pad 4: /flipdot_matrix/R14- -> GND
- Q25 pad 5: /flipdot_matrix/ROW14- -> /flipdot_matrix/ROW16-
- Q25 pad 6: GND -> /flipdot_matrix/R16-
- Q28 pad 1: /flipdot_matrix/R12- -> GND
- Q28 pad 2: /flipdot_matrix/ROW12- -> /flipdot_matrix/ROW10-
- Q28 pad 3: GND -> /flipdot_matrix/R10-
- Q28 pad 4: /flipdot_matrix/R10- -> GND
- Q28 pad 5: /flipdot_matrix/ROW10- -> /flipdot_matrix/ROW12-
- Q28 pad 6: GND -> /flipdot_matrix/R12-
- Q31 pad 1: /flipdot_matrix/R8- -> GND
- Q31 pad 2: /flipdot_matrix/ROW8- -> /flipdot_matrix/ROW6-
- Q31 pad 3: GND -> /flipdot_matrix/R6-
- Q31 pad 4: /flipdot_matrix/R6- -> GND
- Q31 pad 5: /flipdot_matrix/ROW6- -> /flipdot_matrix/ROW8-
- Q31 pad 6: GND -> /flipdot_matrix/R8-
- Q34 pad 1: /flipdot_matrix/R4- -> GND
- Q34 pad 2: /flipdot_matrix/ROW4- -> /flipdot_matrix/ROW2-
- Q34 pad 3: GND -> /flipdot_matrix/R2-
- Q34 pad 4: /flipdot_matrix/R2- -> GND
- Q34 pad 5: /flipdot_matrix/ROW2- -> /flipdot_matrix/ROW4-
- Q34 pad 6: GND -> /flipdot_matrix/R4-
- Q37 pad 1: /flipdot_matrix/R1- -> GND
- Q37 pad 2: /flipdot_matrix/ROW1- -> /flipdot_matrix/ROW3-
- Q37 pad 3: GND -> /flipdot_matrix/R3-
- Q37 pad 4: /flipdot_matrix/R3- -> GND
- Q37 pad 5: /flipdot_matrix/ROW3- -> /flipdot_matrix/ROW1-
- Q37 pad 6: GND -> /flipdot_matrix/R1-
- Q4 pad 1: /flipdot_matrix/FLIP+ -> /flipdot_matrix/R10+
- Q4 pad 2: /flipdot_matrix/ROW12+ -> /flipdot_matrix/ROW10+
- Q4 pad 3: /flipdot_matrix/R12+ -> /flipdot_matrix/FLIP+
- Q4 pad 4: /flipdot_matrix/FLIP+ -> /flipdot_matrix/R12+
- Q4 pad 5: /flipdot_matrix/ROW10+ -> /flipdot_matrix/ROW12+
- Q4 pad 6: /flipdot_matrix/R10+ -> /flipdot_matrix/FLIP+
- Q40 pad 1: /flipdot_matrix/R5- -> GND
- Q40 pad 2: /flipdot_matrix/ROW5- -> /flipdot_matrix/ROW7-
- Q40 pad 3: GND -> /flipdot_matrix/R7-
- Q40 pad 4: /flipdot_matrix/R7- -> GND
- Q40 pad 5: /flipdot_matrix/ROW7- -> /flipdot_matrix/ROW5-
- Q40 pad 6: GND -> /flipdot_matrix/R5-
- Q43 pad 1: /flipdot_matrix/R9- -> GND
- Q43 pad 2: /flipdot_matrix/ROW9- -> /flipdot_matrix/ROW11-
- Q43 pad 3: GND -> /flipdot_matrix/R11-
- Q43 pad 4: /flipdot_matrix/R11- -> GND
- Q43 pad 5: /flipdot_matrix/ROW11- -> /flipdot_matrix/ROW9-
- Q43 pad 6: GND -> /flipdot_matrix/R9-
- Q44 pad 1: /flipdot_matrix/R13- -> GND
- Q44 pad 2: /flipdot_matrix/ROW13- -> /flipdot_matrix/ROW15-
- Q44 pad 3: GND -> /flipdot_matrix/R15-
- Q44 pad 4: /flipdot_matrix/R15- -> GND
- Q44 pad 5: /flipdot_matrix/ROW15- -> /flipdot_matrix/ROW13-
- Q44 pad 6: GND -> /flipdot_matrix/R13-
- Q7 pad 1: /flipdot_matrix/FLIP+ -> /flipdot_matrix/R6+
- Q7 pad 2: /flipdot_matrix/ROW8+ -> /flipdot_matrix/ROW6+
- Q7 pad 3: /flipdot_matrix/R8+ -> /flipdot_matrix/FLIP+
- Q7 pad 4: /flipdot_matrix/FLIP+ -> /flipdot_matrix/R8+
- Q7 pad 5: /flipdot_matrix/ROW6+ -> /flipdot_matrix/ROW8+
- Q7 pad 6: /flipdot_matrix/R6+ -> /flipdot_matrix/FLIP+
- U1 pad 1: /flipdot_matrix/ROW1+ -> /flipdot_matrix/ROW3+
- U1 pad 2: /flipdot_matrix/ROW3+ -> /flipdot_matrix/ROW1+
- U1 pad 21: /flipdot_matrix/ROW2+ -> /flipdot_matrix/ROW4+
- U1 pad 22: /flipdot_matrix/ROW4+ -> /flipdot_matrix/ROW2+
- U1 pad 23: /flipdot_matrix/ROW6+ -> /flipdot_matrix/ROW8+
- U1 pad 24: /flipdot_matrix/ROW8+ -> /flipdot_matrix/ROW6+
- U1 pad 25: /flipdot_matrix/ROW10+ -> /flipdot_matrix/ROW12+
- U1 pad 26: /flipdot_matrix/ROW12+ -> /flipdot_matrix/ROW10+
- U1 pad 27: /flipdot_matrix/ROW14+ -> /flipdot_matrix/ROW16+
- U1 pad 28: /flipdot_matrix/ROW16+ -> /flipdot_matrix/ROW14+
- U1 pad 3: /flipdot_matrix/ROW5+ -> /flipdot_matrix/ROW7+
- U1 pad 4: /flipdot_matrix/ROW7+ -> /flipdot_matrix/ROW5+
- U1 pad 5: /flipdot_matrix/ROW9+ -> /flipdot_matrix/ROW11+
- U1 pad 6: /flipdot_matrix/ROW11+ -> /flipdot_matrix/ROW9+
- U1 pad 7: /flipdot_matrix/ROW13+ -> /flipdot_matrix/ROW15+
- U1 pad 8: /flipdot_matrix/ROW15+ -> /flipdot_matrix/ROW13+
- U3 pad 1: /flipdot_matrix/ROW1- -> /flipdot_matrix/ROW3-
- U3 pad 2: /flipdot_matrix/ROW3- -> /flipdot_matrix/ROW1-
- U3 pad 21: /flipdot_matrix/ROW2- -> /flipdot_matrix/ROW4-
- U3 pad 22: /flipdot_matrix/ROW4- -> /flipdot_matrix/ROW2-
- U3 pad 23: /flipdot_matrix/ROW6- -> /flipdot_matrix/ROW8-
- U3 pad 24: /flipdot_matrix/ROW8- -> /flipdot_matrix/ROW6-
- U3 pad 25: /flipdot_matrix/ROW10- -> /flipdot_matrix/ROW12-
- U3 pad 26: /flipdot_matrix/ROW12- -> /flipdot_matrix/ROW10-
- U3 pad 27: /flipdot_matrix/ROW14- -> /flipdot_matrix/ROW16-
- U3 pad 28: /flipdot_matrix/ROW16- -> /flipdot_matrix/ROW14-
- U3 pad 3: /flipdot_matrix/ROW5- -> /flipdot_matrix/ROW7-
- U3 pad 4: /flipdot_matrix/ROW7- -> /flipdot_matrix/ROW5-
- U3 pad 5: /flipdot_matrix/ROW9- -> /flipdot_matrix/ROW11-
- U3 pad 6: /flipdot_matrix/ROW11- -> /flipdot_matrix/ROW9-
- U3 pad 7: /flipdot_matrix/ROW13- -> /flipdot_matrix/ROW15-
- U3 pad 8: /flipdot_matrix/ROW15- -> /flipdot_matrix/ROW13-
Routing:
- net /flipdot_matrix/ROW11-: track 16.5 -> 9.47 mm
- net /flipdot_matrix/ROW9-: track 9.47 -> 16.5 mm
- net /flipdot_matrix/ROW3-: track 14.0 -> 7.00 mm
- net /flipdot_matrix/ROW1-: track 7.00 -> 14.0 mm
- net /flipdot_matrix/ROW2-: track 27.5 -> 20.6 mm
- net /flipdot_matrix/ROW4-: track 20.6 -> 27.5 mm
- net /flipdot_matrix/ROW7-: track 13.6 -> 7.05 mm
- net /flipdot_matrix/ROW5-: track 7.05 -> 13.6 mm
- net /flipdot_matrix/ROW15-: track 18.8 -> 12.6 mm
- net /flipdot_matrix/ROW13-: track 12.6 -> 18.8 mm
- net /flipdot_matrix/ROW16-: track 27.6 -> 33.7 mm
- net /flipdot_matrix/ROW14-: track 33.7 -> 27.6 mm
- net /flipdot_matrix/ROW8-: track 22.5 -> 28.5 mm
- net /flipdot_matrix/ROW6-: track 28.5 -> 22.5 mm
- net /flipdot_matrix/ROW4+: track 6.18 -> 12.1 mm
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- added copper zone on B.Cu, net GND
- added copper zone on F.Cu, net GND
Other:
- board outline added: 54.6 x 127 mm
- board text added: "AUGUST T 2017 REV1"
