File: driver/_autosave-driver.kicad_pcb (KiCad board)
At the start: 2 copper layers, 59 parts, among them J1 BARREL_JACK, J2 CONN_02X32, Q1 DUAL_NPN_MOSFET, Q10 DUAL_NPN_MOSFET, Q11 DUAL_NPN_MOSFET, Q12 DUAL_NPN_MOSFET, Q13 DUAL_NPN_MOSFET, Q14 DUAL_NPN_MOSFET, Q15 DUAL_NPN_MOSFET, Q16 DUAL_NPN_MOSFET, Q17 DUAL_NPN_MOSFET, Q18 DUAL_NPN_MOSFET, Q19 DUAL_NPN_MOSFET, Q2 DUAL_NPN_MOSFET, Q20 DUAL_NPN_MOSFET, Q21 DUAL_NPN_MOSFET, Q22 DUAL_NPN_MOSFET, Q23 DUAL_NPN_MOSFET, Q24 DUAL_NPN_MOSFET, Q25 DUAL_NPN_MOSFET, Q26 DUAL_NPN_MOSFET, Q27 DUAL_NPN_MOSFET, Q28 DUAL_NPN_MOSFET, Q29 DUAL_NPN_MOSFET, Q3 DUAL_NPN_MOSFET, Q30 DUAL_NPN_MOSFET, Q31 DUAL_NPN_MOSFET, Q32 DUAL_NPN_MOSFET, Q33 DUAL_NPN_MOSFET, Q34 DUAL_NPN_MOSFET, Q35 DUAL_NPN_MOSFET, Q36 DUAL_NPN_MOSFET, Q37 DUAL_NPN_MOSFET, Q38 DUAL_NPN_MOSFET, Q39 DUAL_NPN_MOSFET, Q4 DUAL_NPN_MOSFET, Q40 DUAL_NPN_MOSFET, Q41 DUAL_NPN_MOSFET, Q42 DUAL_NPN_MOSFET, Q43 DUAL_NPN_MOSFET, Q44 DUAL_NPN_MOSFET, Q5 DUAL_NPN_MOSFET, Q6 DUAL_NPN_MOSFET, Q7 DUAL_NPN_MOSFET, Q8 DUAL_NPN_MOSFET, Q9 DUAL_NPN_MOSFET, U1 MCP23017, U2 Teensy3.2, U3 MCP23017, U4 LM7815CT, U5 MCP23017, U6 LF50ABDT-TR, U7 MCP23017, U8 MCP23017, U9 MCP23017

Commit message: more work
Parts:
- U8, U9: moved to B.Cu
- moved U8 28.3 mm to (173.2, 131.1)
- moved U9 22.7 mm to (180.0, 157.2)
- moved Q12 21.1 mm to (158.9, 160.4)
- moved Q24 21.1 mm to (158.9, 170.6)
- moved Q41 21.1 mm to (158.9, 150.2)
- moved Q23 21.1 mm to (158.9, 135.0)
- moved Q11 21.1 mm to (158.9, 124.8)
- moved Q17 21.1 mm to (158.9, 129.9)
- moved Q18 21.1 mm to (158.9, 165.5)
- moved Q29 21.1 mm to (158.9, 140.1)
- moved Q30 21.1 mm to (158.9, 175.6)
- moved Q35 21.1 mm to (158.9, 145.2)
- moved Q36 21.1 mm to (158.9, 180.7)
- moved Q42 21.1 mm to (158.9, 185.8)
- moved Q5 21.1 mm to (158.9, 119.8)
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Connections:
- U8 pad 1: /flipdot_matrix/COL2+ -> /flipdot_matrix/COL8+
- U8 pad 2: /flipdot_matrix/COL2- -> /flipdot_matrix/COL8-
- U8 pad 3: /flipdot_matrix/COL4+ -> /flipdot_matrix/COL6+
- U8 pad 4: /flipdot_matrix/COL4- -> /flipdot_matrix/COL6-
- U8 pad 5: /flipdot_matrix/COL6+ -> /flipdot_matrix/COL4+
- U8 pad 6: /flipdot_matrix/COL6- -> /flipdot_matrix/COL4-
- U8 pad 7: /flipdot_matrix/COL8+ -> /flipdot_matrix/COL2+
- U8 pad 8: /flipdot_matrix/COL8- -> /flipdot_matrix/COL2-
Routing:
- net /flipdot_matrix/COL16+: track 0.00 -> 34.2 mm, vias 0 -> 1
- net /flipdot_matrix/ROW14-: track 0.00 -> 33.7 mm, vias 0 -> 1
- net /flipdot_matrix/COL14+: track 0.00 -> 31.8 mm, vias 0 -> 1
- net /flipdot_matrix/ROW10-: track 0.00 -> 30.9 mm, vias 0 -> 1
- net /flipdot_matrix/COL12+: track 0.00 -> 30.4 mm, vias 0 -> 1
- net /flipdot_matrix/COL16-: track 0.00 -> 29.3 mm, vias 0 -> 1
- net /flipdot_matrix/COL10+: track 0.00 -> 29.2 mm, vias 0 -> 1
- net /flipdot_matrix/ROW6-: track 0.00 -> 28.5 mm, vias 0 -> 1
- net /flipdot_matrix/ROW16-: track 0.00 -> 27.6 mm, vias 0 -> 1
- net /flipdot_matrix/ROW2-: track 0.00 -> 27.5 mm, vias 0 -> 1
- net /flipdot_matrix/COL14-: track 0.00 -> 26.3 mm, vias 0 -> 1
- net /flipdot_matrix/COL2+: track 0.00 -> 26.3 mm, vias 0 -> 1
- net /flipdot_matrix/ROW12-: track 0.00 -> 25.1 mm, vias 0 -> 1
- net /flipdot_matrix/COL12-: track 0.00 -> 24.6 mm, vias 0 -> 1
- net /flipdot_matrix/COL22: track 9.23 -> 33.1 mm
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