File: driver/_saved_driver.sch (KiCad schematic (older format))
At the start: 15 parts, among them J1 BARREL_JACK, J3 CONN_01X04, U1 MCP23017, U2 Teensy3.2, U3 MCP23017, U4 LM7815CT, U5 MCP23017, U6 LF50ABDT-TR, U7 MCP23017, U8 MCP23017, U9 MCP23017

Commit message: done??
probably not
Parts:
- added R2, R3: 4.7k, Resistors_SMD:R_0805_HandSoldering, symbol R
Connections:
- net SCL: now also R2.2
- net SDA: now also R3.2
- net VCC: now also R2.1, R3.1
Changed lines of the file:
@@
 Wire Wire Line
 	14800 15750 14800 15950
+$Comp
+L R R2
+U 1 1 59C84164
+P 21150 4950
+F 0 "R2" V 21230 4950 50  0000 C CNN
+F 1 "4.7k" V 21150 4950 50  0000 C CNN
+F 2 "Resistors_SMD:R_0805_HandSoldering" V 21080 4950 50  0001 C CNN
+F 3 "" H 21150 4950 50  0001 C CNN
+	1    21150 4950
+	0    1    1    0
+$EndComp
+$Comp
+L R R3
+U 1 1 59C844F7
+P 21150 5200
+F 0 "R3" V 21230 5200 50  0000 C CNN
+F 1 "4.7k" V 21150 5200 50  0000 C CNN
+F 2 "Resistors_SMD:R_0805_HandSoldering" V 21080 5200 50  0001 C CNN
+F 3 "" H 21150 5200 50  0001 C CNN
+	1    21150 5200
+	0    1    1    0
+$EndComp
+$Comp
+L VCC #PWR043
+U 1 1 59C849F3
+P 21500 4800
+F 0 "#PWR043" H 21500 4650 50  0001 C CNN
+F 1 "VCC" H 21500 4950 50  0000 C CNN
+F 2 "" H 21500 4800 50  0001 C CNN
+F 3 "" H 21500 4800 50  0001 C CNN
+	1    21500 4800
+	1    0    0    -1
+$EndComp
+Wire Wire Line
+	21300 4950 21500 4950
+Wire Wire Line
+	21500 4800 21500 5200
+Wire Wire Line
+	21500 5200 21300 5200
+Connection ~ 21500 4950
+Wire Wire Line
+	21000 4950 20650 4950
+Wire Wire Line
+	21000 5200 20650 5200
+Text Label 20650 4950 0    60   ~ 0
+SCL
+Text Label 20650 5200 0    60   ~ 0
+SDA
 $EndSCHEMATC

Commit message: fix major goof
Parts:
- C3: footprint Capacitors_SMD:C_0805_HandSoldering -> Resistors_SMD:R_1206_HandSoldering
Connections:
- net flipdot_matrix/ROW1+: now also U1.2 (GPB1); no longer U1.1 (GPB0)
- net flipdot_matrix/ROW1-: now also U3.2 (GPB1); no longer U3.1 (GPB0)
- net flipdot_matrix/ROW10+: now also U1.26 (GPA5); no longer U1.25 (GPA4)
- net flipdot_matrix/ROW10-: now also U3.26 (GPA5); no longer U3.25 (GPA4)
- net flipdot_matrix/ROW11+: now also U1.5 (GPB4); no longer U1.6 (GPB5)
- net flipdot_matrix/ROW11-: now also U3.5 (GPB4); no longer U3.6 (GPB5)
- net flipdot_matrix/ROW12+: now also U1.25 (GPA4); no longer U1.26 (GPA5)
- net flipdot_matrix/ROW12-: now also U3.25 (GPA4); no longer U3.26 (GPA5)
- net flipdot_matrix/ROW13+: now also U1.8 (GPB7); no longer U1.7 (GPB6)
- net flipdot_matrix/ROW13-: now also U3.8 (GPB7); no longer U3.7 (GPB6)
- net flipdot_matrix/ROW14+: now also U1.28 (GPA7); no longer U1.27 (GPA6)
- net flipdot_matrix/ROW14-: now also U3.28 (GPA7); no longer U3.27 (GPA6)
- net flipdot_matrix/ROW15+: now also U1.7 (GPB6); no longer U1.8 (GPB7)
- net flipdot_matrix/ROW15-: now also U3.7 (GPB6); no longer U3.8 (GPB7)
- net flipdot_matrix/ROW16+: now also U1.27 (GPA6); no longer U1.28 (GPA7)
- net flipdot_matrix/ROW16-: now also U3.27 (GPA6); no longer U3.28 (GPA7)
- net flipdot_matrix/ROW2+: now also U1.22 (GPA1); no longer U1.21 (GPA0)
- net flipdot_matrix/ROW2-: now also U3.22 (GPA1); no longer U3.21 (GPA0)
- net flipdot_matrix/ROW3+: now also U1.1 (GPB0); no longer U1.2 (GPB1)
- net flipdot_matrix/ROW3-: now also U3.1 (GPB0); no longer U3.2 (GPB1)
- net flipdot_matrix/ROW4+: now also U1.21 (GPA0); no longer U1.22 (GPA1)
- net flipdot_matrix/ROW4-: now also U3.21 (GPA0); no longer U3.22 (GPA1)
- net flipdot_matrix/ROW5+: now also U1.4 (GPB3); no longer U1.3 (GPB2)
- net flipdot_matrix/ROW5-: now also U3.4 (GPB3); no longer U3.3 (GPB2)
- net flipdot_matrix/ROW6+: now also U1.24 (GPA3); no longer U1.23 (GPA2)
- net flipdot_matrix/ROW6-: now also U3.24 (GPA3); no longer U3.23 (GPA2)
- net flipdot_matrix/ROW7+: now also U1.3 (GPB2); no longer U1.4 (GPB3)
- net flipdot_matrix/ROW7-: now also U3.3 (GPB2); no longer U3.4 (GPB3)
- net flipdot_matrix/ROW8+: now also U1.23 (GPA2); no longer U1.24 (GPA3)
- net flipdot_matrix/ROW8-: now also U3.23 (GPA2); no longer U3.24 (GPA3)
- net flipdot_matrix/ROW9+: now also U1.6 (GPB5); no longer U1.5 (GPB4)
- net flipdot_matrix/ROW9-: now also U3.6 (GPB5); no longer U3.5 (GPB4)
Changed lines of the file:
@@
 F1 "flipdot_matrix.sch" 60
 F2 "FLIP+" I L 7500 4250 60
-F3 "ROW1+" I R 8050 4400 60
-F4 "ROW1-" I R 8050 6000 60
-F5 "ROW2+" I R 8050 5200 60
-F6 "ROW2-" I R 8050 6800 60
-F7 "ROW3+" I R 8050 4500 60
-F8 "ROW4+" I R 8050 5300 60
-F9 "ROW3-" I R 8050 6100 60
-F10 "ROW4-" I R 8050 6900 60
-F11 "ROW5-" I R 8050 6200 60
-F12 "ROW5+" I R 8050 4600 60
-F13 "ROW6+" I R 8050 5400 60
-F14 "ROW6-" I R 8050 7000 60
-F15 "ROW7-" I R 8050 6300 60
-F16 "ROW7+" I R 8050 4700 60
-F17 "ROW8-" I R 8050 7100 60
-F18 "ROW8+" I R 8050 5500 60
-F19 "ROW9+" I R 8050 4800 60
-F20 "ROW9-" I R 8050 6400 60
-F21 "ROW10-" I R 8050 7200 60
-F22 "ROW11-" I R 8050 6500 60
-F23 "ROW10+" I R 8050 5600 60
-F24 "ROW11+" I R 8050 4900 60
-F25 "ROW12+" I R 8050 5700 60
-F26 "ROW12-" I R 8050 7300 60
-F27 "ROW13+" I R 8050 5000 60
-F28 "ROW14+" I R 8050 5800 60
-F29 "ROW15+" I R 8050 5100 60
-F30 "ROW16+" I R 8050 5900 60
-F31 "ROW13-" I R 8050 6600 60
-F32 "ROW14-" I R 8050 7400 60
-F33 "ROW15-" I R 8050 6700 60
-F34 "ROW16-" I R 8050 7500 60
+F3 "ROW1+" I R 8050 4500 60
+F4 "ROW1-" I R 8050 6100 60
+F5 "ROW2+" I R 8050 5300 60
+F6 "ROW2-" I R 8050 6900 60
+F7 "ROW3+" I R 8050 4400 60
+F8 "ROW4+" I R 8050 5200 60
+F9 "ROW3-" I R 8050 6000 60
+F10 "ROW4-" I R 8050 6800 60
+F11 "ROW5-" I R 8050 6300 60
+F12 "ROW5+" I R 8050 4700 60
+F13 "ROW6+" I R 8050 5500 60
+F14 "ROW6-" I R 8050 7100 60
+F15 "ROW7-" I R 8050 6200 60
+F16 "ROW7+" I R 8050 4600 60
+F17 "ROW8-" I R 8050 7000 60
+F18 "ROW8+" I R 8050 5400 60
+F19 "ROW9+" I R 8050 4900 60
+F20 "ROW9-" I R 8050 6500 60
+F21 "ROW10-" I R 8050 7300 60
+F22 "ROW11-" I R 8050 6400 60
+F23 "ROW10+" I R 8050 5700 60
+F24 "ROW11+" I R 8050 4800 60
+F25 "ROW12+" I R 8050 5600 60
+F26 "ROW12-" I R 8050 7200 60
+F27 "ROW13+" I R 8050 5100 60
+F28 "ROW14+" I R 8050 5900 60
+F29 "ROW15+" I R 8050 5000 60
+F30 "ROW16+" I R 8050 5800 60
+F31 "ROW13-" I R 8050 6700 60
+F32 "ROW14-" I R 8050 7500 60
+F33 "ROW15-" I R 8050 6600 60
+F34 "ROW16-" I R 8050 7400 60
 F35 "COL1+" I R 8050 8200 60
 F36 "COL1-" I R 8050 8300 60
@@
 F 0 "C3" H 19625 6750 50  0000 L CNN
 F 1 "22uF" H 19625 6550 50  0000 L CNN
-F 2 "Capacitors_SMD:C_0805_HandSoldering" H 19638 6500 50  0001 C CNN
+F 2 "Resistors_SMD:R_1206_HandSoldering" H 19638 6500 50  0001 C CNN
 F 3 "" H 19600 6650 50  0001 C CNN
 	1    19600 6650
