File: driver/driver.sch (KiCad schematic (older format))
At the start: 14 parts, among them J1 BARREL_JACK, U1 MCP23017, U2 Teensy3.2, U3 MCP23017, U4 LM7815CT, U5 MCP23017, U6 LF50ABDT-TR, U7 MCP23017, U8 MCP23017, U9 MCP23017

Commit message: lots of revs
Connections:
- net flipdot_matrix/COL1+: now also U5.7 (GPB6); no longer U5.1 (GPB0)
- net flipdot_matrix/COL1-: now also U5.8 (GPB7); no longer U5.2 (GPB1)
- net flipdot_matrix/COL17+: now also U7.21 (GPA0); no longer U7.1 (GPB0)
- net flipdot_matrix/COL17-: now also U7.22 (GPA1); no longer U7.2 (GPB1)
- net flipdot_matrix/COL19+: now also U7.23 (GPA2); no longer U7.3 (GPB2)
- net flipdot_matrix/COL19-: now also U7.24 (GPA3); no longer U7.4 (GPB3)
- net flipdot_matrix/COL21+: now also U7.25 (GPA4); no longer U7.5 (GPB4)
- net flipdot_matrix/COL21-: now also U7.26 (GPA5); no longer U7.6 (GPB5)
- net flipdot_matrix/COL25+: now also U7.1 (GPB0); no longer U7.21 (GPA0)
- net flipdot_matrix/COL25-: now also U7.2 (GPB1); no longer U7.22 (GPA1)
- net flipdot_matrix/COL27+: now also U7.3 (GPB2); no longer U7.23 (GPA2)
- net flipdot_matrix/COL27-: now also U7.4 (GPB3); no longer U7.24 (GPA3)
- net flipdot_matrix/COL3+: now also U5.5 (GPB4); no longer U5.3 (GPB2)
- net flipdot_matrix/COL3-: now also U5.6 (GPB5); no longer U5.4 (GPB3)
- net flipdot_matrix/COL5+: now also U5.4 (GPB3); no longer U5.5 (GPB4)
- net flipdot_matrix/COL5-: now also U5.3 (GPB2); no longer U5.6 (GPB5)
- net flipdot_matrix/COL7+: now also U5.2 (GPB1); no longer U5.7 (GPB6)
- net flipdot_matrix/COL7-: now also U5.1 (GPB0); no longer U5.8 (GPB7)
- net flipdot_matrix/ROW1-: now also U3.8 (GPB7); no longer U1.2 (GPB1)
- net flipdot_matrix/ROW10+: now also U1.25 (GPA4); no longer U3.3 (GPB2)
- net flipdot_matrix/ROW10-: now also U3.25 (GPA4); no longer U3.4 (GPB3)
- net flipdot_matrix/ROW11+: now also U1.6 (GPB5); no longer U3.5 (GPB4)
- net flipdot_matrix/ROW11-: now also U3.3 (GPB2); no longer U3.6 (GPB5)
- net flipdot_matrix/ROW12+: now also U1.26 (GPA5); no longer U3.7 (GPB6)
- net flipdot_matrix/ROW12-: now also U3.26 (GPA5); no longer U3.8 (GPB7)
- net flipdot_matrix/ROW13+: now also U1.7 (GPB6); no longer U3.21 (GPA0)
- net flipdot_matrix/ROW13-: now also U3.2 (GPB1); no longer U3.22 (GPA1)
- net flipdot_matrix/ROW14+: now also U1.27 (GPA6); no longer U3.23 (GPA2)
- net flipdot_matrix/ROW14-: now also U3.27 (GPA6); no longer U3.24 (GPA3)
- net flipdot_matrix/ROW15+: now also U1.8 (GPB7); no longer U3.25 (GPA4)
- net flipdot_matrix/ROW15-: now also U3.1 (GPB0); no longer U3.26 (GPA5)
- net flipdot_matrix/ROW16+: now also U1.28 (GPA7); no longer U3.27 (GPA6)
- net flipdot_matrix/ROW2+: now also U1.21 (GPA0); no longer U1.3 (GPB2)
- net flipdot_matrix/ROW2-: now also U3.21 (GPA0); no longer U1.4 (GPB3)
- net flipdot_matrix/ROW3+: now also U1.2 (GPB1); no longer U1.5 (GPB4)
- net flipdot_matrix/ROW3-: now also U3.7 (GPB6); no longer U1.6 (GPB5)
- net flipdot_matrix/ROW4+: now also U1.22 (GPA1); no longer U1.7 (GPB6)
- net flipdot_matrix/ROW4-: now also U3.22 (GPA1); no longer U1.8 (GPB7)
- net flipdot_matrix/ROW5+: now also U1.3 (GPB2); no longer U1.21 (GPA0)
- net flipdot_matrix/ROW5-: now also U3.6 (GPB5); no longer U1.22 (GPA1)
- net flipdot_matrix/ROW6-: now also U3.23 (GPA2); no longer U1.24 (GPA3)
- net flipdot_matrix/ROW7+: now also U1.4 (GPB3); no longer U1.25 (GPA4)
- net flipdot_matrix/ROW7-: now also U3.5 (GPB4); no longer U1.26 (GPA5)
- net flipdot_matrix/ROW8+: now also U1.24 (GPA3); no longer U1.27 (GPA6)
- net flipdot_matrix/ROW8-: now also U3.24 (GPA3); no longer U1.28 (GPA7)
- net flipdot_matrix/ROW9+: now also U1.5 (GPB4); no longer U3.1 (GPB0)
- net flipdot_matrix/ROW9-: now also U3.4 (GPB3); no longer U3.2 (GPB1)
Changed lines of the file:
@@
 F2 "FLIP+" I L 7500 4250 60
 F3 "ROW1+" I R 8050 4400 60
-F4 "ROW1-" I R 8050 4500 60
-F5 "ROW2+" I R 8050 4600 60
-F6 "ROW2-" I R 8050 4700 60
-F7 "ROW3+" I R 8050 4800 60
-F8 "ROW4+" I R 8050 5000 60
-F9 "ROW3-" I R 8050 4900 60
-F10 "ROW4-" I R 8050 5100 60
-F11 "ROW5-" I R 8050 5300 60
-F12 "ROW5+" I R 8050 5200 60
+F4 "ROW1-" I R 8050 6700 60
+F5 "ROW2+" I R 8050 5200 60
+F6 "ROW2-" I R 8050 6800 60
+F7 "ROW3+" I R 8050 4500 60
+F8 "ROW4+" I R 8050 5300 60
+F9 "ROW3-" I R 8050 6600 60
+F10 "ROW4-" I R 8050 6900 60
+F11 "ROW5-" I R 8050 6500 60
+F12 "ROW5+" I R 8050 4600 60
 F13 "ROW6+" I R 8050 5400 60
-F14 "ROW6-" I R 8050 5500 60
-F15 "ROW7-" I R 8050 5700 60
-F16 "ROW7+" I R 8050 5600 60
-F17 "ROW8-" I R 8050 5900 60
-F18 "ROW8+" I R 8050 5800 60
-F19 "ROW9+" I R 8050 6000 60
-F20 "ROW9-" I R 8050 6100 60
-F21 "ROW10-" I R 8050 6300 60
-F22 "ROW11-" I R 8050 6500 60
-F23 "ROW10+" I R 8050 6200 60
-F24 "ROW11+" I R 8050 6400 60
-F25 "ROW12+" I R 8050 6600 60
-F26 "ROW12-" I R 8050 6700 60
-F27 "ROW13+" I R 8050 6800 60
-F28 "ROW14+" I R 8050 7000 60
-F29 "ROW15+" I R 8050 7200 60
-F30 "ROW16+" I R 8050 7400 60
-F31 "ROW13-" I R 8050 6900 60
-F32 "ROW14-" I R 8050 7100 60
-F33 "ROW15-" I R 8050 7300 60
+F14 "ROW6-" I R 8050 7000 60
+F15 "ROW7-" I R 8050 6400 60
+F16 "ROW7+" I R 8050 4700 60
+F17 "ROW8-" I R 8050 7100 60
+F18 "ROW8+" I R 8050 5500 60
+F19 "ROW9+" I R 8050 4800 60
+F20 "ROW9-" I R 8050 6300 60
+F21 "ROW10-" I R 8050 7200 60
+F22 "ROW11-" I R 8050 6200 60
+F23 "ROW10+" I R 8050 5600 60
+F24 "ROW11+" I R 8050 4900 60
+F25 "ROW12+" I R 8050 5700 60
+F26 "ROW12-" I R 8050 7300 60
+F27 "ROW13+" I R 8050 5000 60
+F28 "ROW14+" I R 8050 5800 60
+F29 "ROW15+" I R 8050 5100 60
+F30 "ROW16+" I R 8050 5900 60
+F31 "ROW13-" I R 8050 6100 60
+F32 "ROW14-" I R 8050 7400 60
+F33 "ROW15-" I R 8050 6000 60
 F34 "ROW16-" I R 8050 7500 60
-F35 "COL1+" I R 8050 7600 60
-F36 "COL1-" I R 8050 7700 60
+F35 "COL1+" I R 8050 8200 60
+F36 "COL1-" I R 8050 8300 60
 F37 "COL2+" I R 8050 10800 60
 F38 "COL2-" I R 8050 10900 60
-F39 "COL3+" I R 8050 7800 60
+F39 "COL3+" I R 8050 8000 60
 F40 "COL4+" I R 8050 11000 60
-F41 "COL3-" I R 8050 7900 60
+F41 "COL3-" I R 8050 8100 60
 F42 "COL4-" I R 8050 11100 60
-F43 "COL5-" I R 8050 8100 60
-F44 "COL5+" I R 8050 8000 60
+F43 "COL5-" I R 8050 7800 60
+F44 "COL5+" I R 8050 7900 60
 F45 "COL6+" I R 8050 11200 60
 F46 "COL6-" I R 8050 11300 60
-F47 "COL7-" I R 8050 8300 60
-F48 "COL7+" I R 8050 8200 60
+F47 "COL7-" I R 8050 7600 60
+F48 "COL7+" I R 8050 7700 60
 F49 "COL8-" I R 8050 11500 60
 F50 "COL8+" I R 8050 11400 60
@@
 F65 "COL16+" I R 8050 12200 60
 F66 "COL16-" I R 8050 12300 60
-F67 "COL17+" I R 8050 9200 60
+F67 "COL17+" I R 8050 10000 60
 F68 "COL18+" I R 8050 12400 60
-F69 "COL17-" I R 8050 9300 60
+F69 "COL17-" I R 8050 10100 60
 F70 "COL18-" I R 8050 12500 60
-F71 "COL19-" I R 8050 9500 60
-F72 "COL19+" I R 8050 9400 60
+F71 "COL19-" I R 8050 10300 60
+F72 "COL19+" I R 8050 10200 60
 F73 "COL20+" I R 8050 12600 60
 F74 "COL20-" I R 8050 12700 60
-F75 "COL21-" I R 8050 9700 60
-F76 "COL21+" I R 8050 9600 60
+F75 "COL21-" I R 8050 10500 60
+F76 "COL21+" I R 8050 10400 60
 F77 "COL22-" I R 8050 12900 60
 F78 "COL22+" I R 8050 12800 60
@@
 F80 "COL23-" I R 8050 9900 60
 F81 "COL24-" I R 8050 13100 60
-F82 "COL25-" I R 8050 10100 60
+F82 "COL25-" I R 8050 9300 60
 F83 "COL24+" I R 8050 13000 60
-F84 "COL25+" I R 8050 10000 60
+F84 "COL25+" I R 8050 9200 60
 F85 "COL26+" I R 8050 13200 60
 F86 "COL26-" I R 8050 13300 60
-F87 "COL27+" I R 8050 10200 60
+F87 "COL27+" I R 8050 9400 60
 F88 "COL28+" I R 8050 13400 60
-F89 "COL27-" I R 8050 10300 60
+F89 "COL27-" I R 8050 9500 60
 F90 "COL28-" I R 8050 13500 60
 $EndSheet
@@
 Wire Wire Line
 	13700 9500 8050 9500
-Wire Wire Line
-	8050 9600 13700 9600
-Wire Wire Line
-	13700 9700 8050 9700
 Wire Wire Line
 	8050 9800 13700 9800
@@
 Text Notes 13950 5700 2    60   ~ 0
 ROW CHIP!
-NoConn ~ 13700 10500
-NoConn ~ 13700 10600
 NoConn ~ 13700 10700
 NoConn ~ 13700 10800
@@
 Wire Wire Line
 	10550 13500 8050 13500
+NoConn ~ 13700 9600
+NoConn ~ 13700 9700
+Wire Wire Line
+	8050 10400 13450 10400
+Wire Wire Line
+	13450 10400 13450 10500
+Wire Wire Line
+	13450 10500 13700 10500
+Wire Wire Line
+	13700 10600 13350 10600
+Wire Wire Line
+	13350 10600 13350 10500
+Wire Wire Line
+	13350 10500 8050 10500
 $EndSCHEMATC

Commit message: more work
Connections:
- net flipdot_matrix/COL2+: now also U8.7 (GPB6); no longer U8.1 (GPB0)
- net flipdot_matrix/COL2-: now also U8.8 (GPB7); no longer U8.2 (GPB1)
- net flipdot_matrix/COL4+: now also U8.5 (GPB4); no longer U8.3 (GPB2)
- net flipdot_matrix/COL4-: now also U8.6 (GPB5); no longer U8.4 (GPB3)
- net flipdot_matrix/COL6+: now also U8.3 (GPB2); no longer U8.5 (GPB4)
- net flipdot_matrix/COL6-: now also U8.4 (GPB3); no longer U8.6 (GPB5)
- net flipdot_matrix/COL8+: now also U8.1 (GPB0); no longer U8.7 (GPB6)
- net flipdot_matrix/COL8-: now also U8.2 (GPB1); no longer U8.8 (GPB7)
- net flipdot_matrix/ROW1-: now also U3.1 (GPB0); no longer U3.8 (GPB7)
- net flipdot_matrix/ROW11-: now also U3.6 (GPB5); no longer U3.3 (GPB2)
- net flipdot_matrix/ROW13-: now also U3.7 (GPB6); no longer U3.2 (GPB1)
- net flipdot_matrix/ROW15-: now also U3.8 (GPB7); no longer U3.1 (GPB0)
- net flipdot_matrix/ROW3-: now also U3.2 (GPB1); no longer U3.7 (GPB6)
- net flipdot_matrix/ROW5-: now also U3.3 (GPB2); no longer U3.6 (GPB5)
- net flipdot_matrix/ROW7-: now also U3.4 (GPB3); no longer U3.5 (GPB4)
- net flipdot_matrix/ROW9-: now also U3.5 (GPB4); no longer U3.4 (GPB3)
Changed lines of the file:
@@
 F2 "FLIP+" I L 7500 4250 60
 F3 "ROW1+" I R 8050 4400 60
-F4 "ROW1-" I R 8050 6700 60
+F4 "ROW1-" I R 8050 6000 60
 F5 "ROW2+" I R 8050 5200 60
 F6 "ROW2-" I R 8050 6800 60
 F7 "ROW3+" I R 8050 4500 60
 F8 "ROW4+" I R 8050 5300 60
-F9 "ROW3-" I R 8050 6600 60
+F9 "ROW3-" I R 8050 6100 60
 F10 "ROW4-" I R 8050 6900 60
-F11 "ROW5-" I R 8050 6500 60
+F11 "ROW5-" I R 8050 6200 60
 F12 "ROW5+" I R 8050 4600 60
 F13 "ROW6+" I R 8050 5400 60
 F14 "ROW6-" I R 8050 7000 60
-F15 "ROW7-" I R 8050 6400 60
+F15 "ROW7-" I R 8050 6300 60
 F16 "ROW7+" I R 8050 4700 60
 F17 "ROW8-" I R 8050 7100 60
 F18 "ROW8+" I R 8050 5500 60
 F19 "ROW9+" I R 8050 4800 60
-F20 "ROW9-" I R 8050 6300 60
+F20 "ROW9-" I R 8050 6400 60
 F21 "ROW10-" I R 8050 7200 60
-F22 "ROW11-" I R 8050 6200 60
+F22 "ROW11-" I R 8050 6500 60
 F23 "ROW10+" I R 8050 5600 60
 F24 "ROW11+" I R 8050 4900 60
@@
 F29 "ROW15+" I R 8050 5100 60
 F30 "ROW16+" I R 8050 5900 60
-F31 "ROW13-" I R 8050 6100 60
+F31 "ROW13-" I R 8050 6600 60
 F32 "ROW14-" I R 8050 7400 60
-F33 "ROW15-" I R 8050 6000 60
+F33 "ROW15-" I R 8050 6700 60
 F34 "ROW16-" I R 8050 7500 60
 F35 "COL1+" I R 8050 8200 60
 F36 "COL1-" I R 8050 8300 60
-F37 "COL2+" I R 8050 10800 60
-F38 "COL2-" I R 8050 10900 60
+F37 "COL2+" I R 8050 11400 60
+F38 "COL2-" I R 8050 11500 60
 F39 "COL3+" I R 8050 8000 60
-F40 "COL4+" I R 8050 11000 60
+F40 "COL4+" I R 8050 11200 60
 F41 "COL3-" I R 8050 8100 60
-F42 "COL4-" I R 8050 11100 60
+F42 "COL4-" I R 8050 11300 60
 F43 "COL5-" I R 8050 7800 60
 F44 "COL5+" I R 8050 7900 60
-F45 "COL6+" I R 8050 11200 60
-F46 "COL6-" I R 8050 11300 60
+F45 "COL6+" I R 8050 11000 60
+F46 "COL6-" I R 8050 11100 60
 F47 "COL7-" I R 8050 7600 60
 F48 "COL7+" I R 8050 7700 60
-F49 "COL8-" I R 8050 11500 60
-F50 "COL8+" I R 8050 11400 60
+F49 "COL8-" I R 8050 10900 60
+F50 "COL8+" I R 8050 10800 60
 F51 "COL9+" I R 8050 8400 60
 F52 "COL9-" I R 8050 8500 60

Commit message: closer to final
Parts:
- added J3: CONN_01X04, Pin_Headers:Pin_Header_Straight_1x04_Pitch2.54mm, symbol CONN_01X04
- C1, C2: footprint Capacitors_THT:CP_Radial_Tantal_D10.5mm_P5.00mm -> Capacitors_SMD:C_0805_HandSoldering
- C3: value 10uF -> 22uF; footprint Capacitors_THT:CP_Radial_Tantal_D10.5mm_P5.00mm -> Capacitors_SMD:C_0805_HandSoldering
- R1: footprint (none) -> Resistors_THT:R_Axial_DIN0414_L11.9mm_D4.5mm_P15.24mm_Horizontal
Connections:
- net GND: now also J3.4 (P4)
- net SCL: now also J3.2 (P2)
- net SDA: now also J3.3 (P3)
- net VCC: now also J3.1 (P1)
- net flipdot_matrix/COL18+: now also U9.8 (GPB7); no longer U9.1 (GPB0)
- net flipdot_matrix/COL18-: now also U9.7 (GPB6); no longer U9.2 (GPB1)
- net flipdot_matrix/COL20+: now also U9.6 (GPB5); no longer U9.3 (GPB2)
- net flipdot_matrix/COL20-: now also U9.5 (GPB4); no longer U9.4 (GPB3)
- net flipdot_matrix/COL22+: now also U9.4 (GPB3); no longer U9.5 (GPB4)
- net flipdot_matrix/COL22-: now also U9.3 (GPB2); no longer U9.6 (GPB5)
- net flipdot_matrix/COL23+: now also U7.1 (GPB0); no longer U7.7 (GPB6)
- net flipdot_matrix/COL23-: now also U7.2 (GPB1); no longer U7.8 (GPB7)
- net flipdot_matrix/COL24+: now also U9.24 (GPA3); no longer U9.7 (GPB6)
- net flipdot_matrix/COL24-: now also U9.23 (GPA2); no longer U9.8 (GPB7)
- net flipdot_matrix/COL25+: now also U7.3 (GPB2); no longer U7.1 (GPB0)
- net flipdot_matrix/COL25-: now also U7.4 (GPB3); no longer U7.2 (GPB1)
- net flipdot_matrix/COL26+: now also U9.22 (GPA1); no longer U9.21 (GPA0)
- net flipdot_matrix/COL26-: now also U9.21 (GPA0); no longer U9.22 (GPA1)
- net flipdot_matrix/COL27+: now also U7.7 (GPB6); no longer U7.3 (GPB2)
- net flipdot_matrix/COL27-: now also U7.8 (GPB7); no longer U7.4 (GPB3)
- net flipdot_matrix/COL28+: now also U9.1 (GPB0); no longer U9.23 (GPA2)
- net flipdot_matrix/COL28-: now also U9.2 (GPB1); no longer U9.24 (GPA3)
- net JACK_IN: now reaches C1.1, J1.1, U4.1 (IN), U6.1 (Vin)
Changed lines of the file:
@@
 F66 "COL16-" I R 8050 12300 60
 F67 "COL17+" I R 8050 10000 60
-F68 "COL18+" I R 8050 12400 60
+F68 "COL18+" I R 8050 13100 60
 F69 "COL17-" I R 8050 10100 60
-F70 "COL18-" I R 8050 12500 60
+F70 "COL18-" I R 8050 13000 60
 F71 "COL19-" I R 8050 10300 60
 F72 "COL19+" I R 8050 10200 60
-F73 "COL20+" I R 8050 12600 60
-F74 "COL20-" I R 8050 12700 60
+F73 "COL20+" I R 8050 12900 60
+F74 "COL20-" I R 8050 12800 60
 F75 "COL21-" I R 8050 10500 60
 F76 "COL21+" I R 8050 10400 60
-F77 "COL22-" I R 8050 12900 60
-F78 "COL22+" I R 8050 12800 60
-F79 "COL23+" I R 8050 9800 60
-F80 "COL23-" I R 8050 9900 60
-F81 "COL24-" I R 8050 13100 60
-F82 "COL25-" I R 8050 9300 60
-F83 "COL24+" I R 8050 13000 60
-F84 "COL25+" I R 8050 9200 60
-F85 "COL26+" I R 8050 13200 60
-F86 "COL26-" I R 8050 13300 60
-F87 "COL27+" I R 8050 9400 60
-F88 "COL28+" I R 8050 13400 60
-F89 "COL27-" I R 8050 9500 60
-F90 "COL28-" I R 8050 13500 60
+F77 "COL22-" I R 8050 12600 60
+F78 "COL22+" I R 8050 12700 60
+F79 "COL23+" I R 8050 9200 60
+F80 "COL23-" I R 8050 9300 60
+F81 "COL24-" I R 8050 13400 60
+F82 "COL25-" I R 8050 9500 60
+F83 "COL24+" I R 8050 13500 60
+F84 "COL25+" I R 8050 9400 60
+F85 "COL26+" I R 8050 13300 60
+F86 "COL26-" I R 8050 13200 60
+F87 "COL27+" I R 8050 9800 60
+F88 "COL28+" I R 8050 12400 60
+F89 "COL27-" I R 8050 9900 60
+F90 "COL28-" I R 8050 12500 60
 $EndSheet
 Wire Wire Line
@@
 F 0 "C1" H 19175 8000 50  0000 L CNN
 F 1 "10uF" H 19175 7800 50  0000 L CNN
-F 2 "Capacitors_THT:CP_Radial_Tantal_D10.5mm_P5.00mm" H 19188 7750 50  0001 C CNN
+F 2 "Capacitors_SMD:C_0805_HandSoldering" H 19188 7750 50  0001 C CNN
 F 3 "" H 19150 7900 50  0001 C CNN
 	1    19150 7900
@@
 F 0 "C2" H 20575 8000 50  0000 L CNN
 F 1 "10uF" H 20575 7800 50  0000 L CNN
-F 2 "Capacitors_THT:CP_Radial_Tantal_D10.5mm_P5.00mm" H 20588 7750 50  0001 C CNN
+F 2 "Capacitors_SMD:C_0805_HandSoldering" H 20588 7750 50  0001 C CNN
 F 3 "" H 20550 7900 50  0001 C CNN
 	1    20550 7900
@@
 P 19600 6650
 F 0 "C3" H 19625 6750 50  0000 L CNN
-F 1 "10uF" H 19625 6550 50  0000 L CNN
-F 2 "Capacitors_THT:CP_Radial_Tantal_D10.5mm_P5.00mm" H 19638 6500 50  0001 C CNN
+F 1 "22uF" H 19625 6550 50  0000 L CNN
+F 2 "Capacitors_SMD:C_0805_HandSoldering" H 19638 6500 50  0001 C CNN
 F 3 "" H 19600 6650 50  0001 C CNN
 	1    19600 6650
@@
 F 0 "R1" V 7130 4250 50  0000 C CNN
 F 1 "CURRLIM" V 7050 4250 50  0000 C CNN
-F 2 "" V 6980 4250 50  0001 C CNN
+F 2 "Resistors_THT:R_Axial_DIN0414_L11.9mm_D4.5mm_P15.24mm_Horizontal" V 6980 4250 50  0001 C CNN
 F 3 "" H 7050 4250 50  0001 C CNN
 	1    7050 4250
@@
 Wire Wire Line
 	13350 10500 8050 10500
+$Comp
+L CONN_01X04 J3
+U 1 1 59B906C2
+P 21300 3750
+F 0 "J3" H 21300 4000 50  0000 C CNN
+F 1 "CONN_01X04" V 21400 3750 50  0000 C CNN
+F 2 "Pin_Headers:Pin_Header_Straight_1x04_Pitch2.54mm" H 21300 3750 50  0001 C CNN
+F 3 "" H 21300 3750 50  0001 C CNN
+	1    21300 3750
+	1    0    0    -1
+$EndComp
+Wire Wire Line
+	21100 3600 20800 3600
+Wire Wire Line
+	21100 3700 20800 3700
+Wire Wire Line
+	21100 3800 20800 3800
+Wire Wire Line
+	21100 3900 20800 3900
+Wire Wire Line
+	20800 3600 20800 3450
+Wire Wire Line
+	20800 3900 20800 4050
+$Comp
+L VCC #PWR041
+U 1 1 59B932A1
+P 20800 3450
+F 0 "#PWR041" H 20800 3300 50  0001 C CNN
+F 1 "VCC" H 20800 3600 50  0000 C CNN
+F 2 "" H 20800 3450 50  0001 C CNN
+F 3 "" H 20800 3450 50  0001 C CNN
+	1    20800 3450
+	1    0    0    -1
+$EndComp
+$Comp
+L GND #PWR042
+U 1 1 59B93A6B
+P 20800 4050
+F 0 "#PWR042" H 20800 3800 50  0001 C CNN
+F 1 "GND" H 20800 3900 50  0000 C CNN
+F 2 "" H 20800 4050 50  0001 C CNN
+F 3 "" H 20800 4050 50  0001 C CNN
+	1    20800 4050
+	1    0    0    -1
+$EndComp
+Text Label 20800 3700 0    60   ~ 0
+SCL
+Text Label 20800 3800 0    60   ~ 0
+SDA
+Text Label 18150 7700 0    60   ~ 0
+JACK_IN
 $EndSCHEMATC

Commit message: done??
probably not
Parts:
- added R? (x2): 4.7k, symbol R
Connections:
- net GND: now also U8.16 (A1), U9.16 (A1); no longer U7.15 (A0), U8.17 (A2), U9.15 (A0), U9.17 (A2)
- net SCL: now also R?.2
- net SDA: now also R?.2
- net VCC: now also U7.15 (A0), U8.17 (A2), U9.15 (A0), U9.17 (A2), R?.1, R?.1; no longer U8.16 (A1), U9.16 (A1)
Other:
- note added: "ADDR 0 = 000\n"
- note added: "ADDR 1 = 001"
- note added: "ADDR 2 = 010"
- note added: "ADDR 3 = 011"
- note added: "ADDR 4 = 100"
- note added: "ADDR 5 = 101\n"
- note removed: "ADDR 0\n"
- note removed: "ADDR 1"
- note removed: "ADDR 2"
Changed lines of the file:
@@
 L VCC #PWR029
 U 1 1 5988DC91
-P 14900 15750
-F 0 "#PWR029" H 14900 15600 50  0001 C CNN
-F 1 "VCC" H 14900 15900 50  0000 C CNN
-F 2 "" H 14900 15750 50  0001 C CNN
-F 3 "" H 14900 15750 50  0001 C CNN
-	1    14900 15750
+P 14900 15650
+F 0 "#PWR029" H 14900 15500 50  0001 C CNN
+F 1 "VCC" H 14900 15800 50  0000 C CNN
+F 2 "" H 14900 15650 50  0001 C CNN
+F 3 "" H 14900 15650 50  0001 C CNN
+	1    14900 15650
 	1    0    0    -1
 $EndComp
@@
 	14700 10800 14800 10800
 Wire Wire Line
-	14800 10600 14800 10900
+	14800 10800 14800 10900
 Wire Wire Line
 	14700 10600 14800 10600
 Connection ~ 14800 10800
-Wire Wire Line
-	14700 10700 14900 10700
 Wire Wire Line
 	15300 10300 14700 10300
@@
 	14850 11800 14700 11800
 Wire Wire Line
-	14700 13400 14800 13400
-Wire Wire Line
-	14800 13200 14800 13500
-Wire Wire Line
 	14700 13200 14800 13200
-Connection ~ 14800 13400
-Wire Wire Line
-	14700 13300 14900 13300
 Wire Wire Line
 	15300 12900 14700 12900
@@
 	14850 14250 14700 14250
 Wire Wire Line
-	14700 15850 14800 15850
-Wire Wire Line
-	14800 15650 14800 15950
-Wire Wire Line
-	14700 15650 14800 15650
-Connection ~ 14800 15850
-Wire Wire Line
-	14700 15750 14900 15750
+	14700 15650 14900 15650
 Wire Wire Line
 	15300 15350 14700 15350
@@
 Wire Wire Line
 	6700 4250 6900 4250
-Text Notes 15200 2700 2    60   ~ 0
-ADDR 0\n
-Text Notes 15200 5400 2    60   ~ 0
-ADDR 1
-Text Notes 15250 8250 2    60   ~ 0
-ADDR 2
+Text Notes 15550 2750 2    60   ~ 0
+ADDR 0 = 000\n
+Text Notes 15550 5400 2    60   ~ 0
+ADDR 1 = 001
+Text Notes 15600 8250 2    60   ~ 0
+ADDR 2 = 010
 Wire Wire Line
 	15400 6600 15600 6600
@@
 Text Label 18150 7700 0    60   ~ 0
 JACK_IN
+Text Notes 15000 11000 0    60   ~ 0
+ADDR 3 = 011
+Wire Wire Line
+	14700 10700 14900 10700
+Wire Wire Line
+	14800 10600 14800 10700
+Connection ~ 14800 10700
+Text Notes 15000 13550 0    60   ~ 0
+ADDR 4 = 100
+Wire Wire Line
+	14800 13200 14800 13500
+Wire Wire Line
+	14700 13300 14800 13300
+Connection ~ 14800 13300
+Wire Wire Line
+	14700 13400 14900 13400
+Wire Wire Line
+	14900 13400 14900 13300
+Text Notes 15050 16050 0    60   ~ 0
+ADDR 5 = 101\n
+Wire Wire Line
+	14700 15850 14900 15850
+Wire Wire Line
+	14900 15850 14900 15650
+Wire Wire Line
+	14700 15750 14800 15750
+Wire Wire Line
+	14800 15750 14800 15950
+$Comp
+L R R?
+U 1 1 59C84164
+P 21150 4950
+F 0 "R?" V 21230 4950 50  0000 C CNN
+F 1 "4.7k" V 21150 4950 50  0000 C CNN
+F 2 "" V 21080 4950 50  0001 C CNN
+F 3 "" H 21150 4950 50  0001 C CNN
+	1    21150 4950
+	0    1    1    0
+$EndComp
+$Comp
+L R R?
+U 1 1 59C844F7
+P 21150 5200
+F 0 "R?" V 21230 5200 50  0000 C CNN
+F 1 "4.7k" V 21150 5200 50  0000 C CNN
+F 2 "" V 21080 5200 50  0001 C CNN
+F 3 "" H 21150 5200 50  0001 C CNN
+	1    21150 5200
+	0    1    1    0
+$EndComp
+$Comp
+L VCC #PWR?
+U 1 1 59C849F3
+P 21500 4800
+F 0 "#PWR?" H 21500 4650 50  0001 C CNN
+F 1 "VCC" H 21500 4950 50  0000 C CNN
+F 2 "" H 21500 4800 50  0001 C CNN
+F 3 "" H 21500 4800 50  0001 C CNN
+	1    21500 4800
+	1    0    0    -1
+$EndComp
+Wire Wire Line
+	21300 4950 21500 4950
+Wire Wire Line
+	21500 4800 21500 5200
+Wire Wire Line
+	21500 5200 21300 5200
+Connection ~ 21500 4950
+Wire Wire Line
+	21000 4950 20650 4950
+Wire Wire Line
+	21000 5200 20650 5200
+Text Label 20650 4950 0    60   ~ 0
+SCL
+Text Label 20650 5200 0    60   ~ 0
+SDA
 $EndSCHEMATC
